File: PCB/Slave/Slave1 - Copy/Slave.kicad_pcb (KiCad board)
At the start: 2 copper layers, 97 parts, among them J1 Jack-DC, J11 MH, J12 LED1, J13 LED3, J14 LED5, J15 LED2, J16 LED4, J3 PGM, J4 S1..4, J5 S5..8, J6 S9..12, J8 MH, J9 MH, Q1 Q_PMOS_GSD, Q10 Q_PMOS_GSD, Q11 Q_PMOS_GSD, Q12 Q_PMOS_GSD, Q2 Q_PMOS_GSD, Q3 Q_PMOS_GSD, Q4 Q_PMOS_GSD, Q5 Q_PMOS_GSD, Q6 Q_PMOS_GSD, Q7 Q_PMOS_GSD, Q8 Q_PMOS_GSD, Q9 Q_PMOS_GSD, SW1 SW_Push, U1 MCP23S17, U2 LT3080, U3 dsPIC33EPXXXGP502, U4 PCA9745B, U5 nRF24L01+

Commit message: working on the pcb
Parts:
- added C10: 1µ, Capacitors_SMD:C_0603_HandSoldering, F.Cu at (200.2, 141.8)
- added C2: 1µ, Capacitors_SMD:C_0603_HandSoldering, F.Cu at (221.2, 116.5)
- added J10: MH, Mounting_Holes:MountingHole_2.7mm_M2.5_ISO14580_Pad, F.Cu at (204.1, 108.4)
- added J2: GP_IO, Pin_Headers:Pin_Header_Straight_1x04_Pitch2.54mm, F.Cu at (58.0, 137.0)
- added J7: PIC_IO, Pin_Headers:Pin_Header_Straight_1x05_Pitch2.54mm, F.Cu at (165.4, 107.4)
- moved J11 235.9 mm to (209.6, 108.4)
- moved J8 234.2 mm to (199.5, 122.7)
- moved J13 166.6 mm to (214.5, 108.4), turned to 0 degrees
- moved D1 154.2 mm to (221.4, 106.6), turned to 0 degrees
- moved R6 153.9 mm to (221.4, 111.6)
- moved J12 152.5 mm to (204.4, 116.9), turned to 0 degrees
- moved C9 150.0 mm to (209.9, 132.8)
- moved C3 150.0 mm to (217.1, 114.2), turned to 0 degrees
- moved R5 148.3 mm to (208.8, 122.9), turned to 0 degrees
- moved J15 146.4 mm to (199.0, 131.2), turned to 0 degrees
- moved C7 146.1 mm to (205.8, 132.8)
- moved C1 145.1 mm to (213.0, 122.1), turned to 0 degrees
- moved R1 144.0 mm to (210.3, 128.0), turned to 0 degrees
- moved R4 138.1 mm to (205.9, 128.0), turned to 0 degrees
- moved C6 137.7 mm to (200.2, 137.0), turned to 0 degrees
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Connections:
- D2 pad 1: GND -> Net-(D2-Pad1)
- R3 pad 2: Net-(D2-Pad2) -> Net-(R3-Pad2)
- U3 pad 10: Net-(U3-Pad10) -> /IO4
- U3 pad 12: Net-(U3-Pad12) -> /IO5
- U3 pad 2: Net-(U3-Pad2) -> /IO1
- U3 pad 3: Net-(U3-Pad3) -> /IO2
- U3 pad 9: Net-(U3-Pad9) -> /IO3
- U4 pad 12: /R2 -> /B2
- U4 pad 13: /B3 -> /R3
- U4 pad 15: /R3 -> /B3
- U4 pad 16: /B4 -> /R4
- U4 pad 18: /R4 -> /B4
- U4 pad 20: /B5 -> /R5
- U4 pad 22: /R5 -> /B5
- U4 pad 6: /B1 -> /R1
- U4 pad 8: /R1 -> /B1
- U4 pad 9: /B2 -> /R2
Routing:
- net /R5: track 32.9 -> 0.00 mm
- net /G5: track 30.0 -> 0.00 mm
- net /B5: track 27.2 -> 0.00 mm
- net /R4: track 26.8 -> 0.00 mm
- net /NRF_MOSI: track 24.9 -> 0.00 mm
- net /G4: track 24.2 -> 0.00 mm
- net /B1: track 23.6 -> 0.00 mm
- net /G1: track 23.2 -> 0.00 mm
- net /R1: track 22.3 -> 0.00 mm
- net /B4: track 21.4 -> 0.00 mm
- net /R3: track 20.8 -> 0.00 mm
- net /B2: track 19.1 -> 0.00 mm
- net /G2: track 18.9 -> 0.00 mm
- net /NRF_CSN: track 18.7 -> 0.00 mm
- net /R2: track 18.2 -> 0.00 mm
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