File: PCB/Slave/Slave1 - Copy/Slave.sch (KiCad schematic (older format))
At the start: 39 parts, among them J1 Jack-DC, J10 MH, J11 MH, J12 LED1, J13 LED3, J14 LED5, J15 LED2, J16 LED4, J3 PGM, J4 S1..4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

Commit message: working on the pcb
Parts:
- added C10, C2: 1µ, Capacitors_SMD:C_0603_HandSoldering, symbol C
- added J2: GP_IO, Pin_Headers:Pin_Header_Straight_1x04_Pitch2.54mm, symbol Conn_01x04
Connections:
- net +3V3: now also C10.1, C2.1
- net B1: now also U4.8 (LED2); no longer U4.6 (LED0)
- net B2: now also U4.12 (LED5); no longer U4.9 (LED3)
- net B3: now also U4.15 (LED8); no longer U4.13 (LED6)
- net B4: now also U4.18 (LED11); no longer U4.16 (LED9)
- net B5: now also U4.22 (LED14); no longer U4.20 (LED12)
- net GND: now also C10.2, C2.2; no longer D2.1 (K)
- net R1: now also U4.6 (LED0); no longer U4.8 (LED2)
- net R2: now also U4.9 (LED3); no longer U4.12 (LED5)
- net R3: now also U4.13 (LED6); no longer U4.15 (LED8)
- net R4: now also U4.16 (LED9); no longer U4.18 (LED11)
- net R5: now also U4.20 (LED12); no longer U4.22 (LED14)
- net at U1.25 (GPA4): now also J2.1 (Pin_1)
- net at U1.26 (GPA5): now also J2.2 (Pin_2)
- net at U1.27 (GPA6): now also J2.3 (Pin_3)
- net at U1.28 (GPA7): now also J2.4 (Pin_4)
- net at R3.2: no longer D2.2 (A)
- no-connect marks 10 -> 6
Other:
- moved on the sheet: J12, J13, J14, J15, J16
