File: PCB/Slave/Slave1/PMOS_ARRAY.sch (KiCad schematic (older format))
At the start: 60 parts, among them Q1 Q_PMOS_GSD, Q10 Q_PMOS_GSD, Q11 Q_PMOS_GSD, Q12 Q_PMOS_GSD, Q2 Q_PMOS_GSD, Q3 Q_PMOS_GSD, Q4 Q_PMOS_GSD, Q5 Q_PMOS_GSD, Q6 Q_PMOS_GSD, Q7 Q_PMOS_GSD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

Commit message: updated pcb for prototype
Parts:
- added C10, C12, C13, C14, C15, C16, C17, C18, C19, C2, C20, C21: 1µ, Capacitors_SMD:C_0603_HandSoldering, symbol C
Connections:
- net GND: now also C10.2, C12.2, C13.2, C14.2, C15.2, C16.2, C17.2, C18.2, C19.2, C2.2, C20.2, C21.2
- net S1: now also C2.1
- net S10: now also C19.1
- net S11: now also C20.1
- net S12: now also C21.1
- net S2: now also C10.1
- net S3: now also C12.1
- net S4: now also C13.1
- net S5: now also C14.1
- net S6: now also C15.1
- net S7: now also C16.1
- net S8: now also C17.1
- net S9: now also C18.1
- net +3V3 renamed Vdd
