File: PCB/Slave/Slave1/Slave.kicad_pcb (KiCad board)
At the start: 2 copper layers, 56 x 61.5 mm, 95 parts, among them J1 Jack-DC, J12 LED1, J13 LED3, J14 LED5, J15 LED2, J16 LED4, J3 PGM, J4 S1..4, J5 S5..8, J6 S9..12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

Commit message: better slave pcb
Parts:
- added D16: D, Diodes_SMD:D_MicroMELF_Hadsoldering, F.Cu at (64.0, 118.5)
- added D17: LED, LEDs:LED_0603_HandSoldering, F.Cu at (70.5, 126.0)
- added J2: PPIO, Pin_Headers:Pin_Header_Straight_1x04_Pitch2.54mm, F.Cu at (84.5, 164.0)
- added J7: MH, Mounting_Holes:MountingHole_2.7mm_M2.5_ISO14580_Pad, F.Cu at (61.0, 163.0)
- added R43: 2.2k, Resistors_SMD:R_0603_HandSoldering, F.Cu at (70.5, 124.0)
- moved J9 34.4 mm to (61.0, 131.0)
- moved C9 12.1 mm to (65.0, 116.0), turned to 180 degrees
- moved D3 5.10 mm to (73.5, 156.5)
- moved C6 4.12 mm to (63.0, 121.0), turned to 0 degrees
- moved C8 4.12 mm to (65.0, 129.0), turned to 90 degrees
- moved R1 3.64 mm to (70.5, 114.0)
- moved J12 3.50 mm to (56.5, 135.0)
- moved J13 3.50 mm to (56.5, 149.0)
- moved J14 3.50 mm to (56.5, 163.0)
- moved J15 3.50 mm to (56.5, 142.0)
- moved J16 3.50 mm to (56.5, 156.0)
- moved R5 3.50 mm to (65.5, 144.5)
- moved U4 3.50 mm to (68.5, 152.0)
- moved U2 3.35 mm to (59.0, 126.5)
- moved U3 3.20 mm to (79.5, 124.0)
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Routing:
- net Net-(C6-Pad1): track 20.6 -> 4.05 mm
- net Net-(J2-Pad1): track 0.00 -> 14.6 mm, vias 0 -> 1
- net Net-(J2-Pad2): track 0.00 -> 12.3 mm, vias 0 -> 1
- net /R4: track 26.8 -> 15.8 mm, vias 0 -> 2
- net Net-(J2-Pad3): track 0.00 -> 9.86 mm
- net /G4: track 24.2 -> 16.9 mm, vias 0 -> 2
- net /B5: track 27.2 -> 20.0 mm
- net /R5: track 32.9 -> 26.2 mm
- net Net-(J2-Pad4): track 0.00 -> 6.69 mm
- net /R3: track 20.8 -> 27.3 mm, vias 0 -> 2
- net /G5: track 30.0 -> 23.6 mm
- net /SEL_MISO: track 48.6 -> 54.6 mm
- net /PCA_CS: track 27.6 -> 23.2 mm
- net Net-(R43-Pad1): track 0.00 -> 3.99 mm
- net /RESET: track 62.9 -> 58.9 mm, vias 6 -> 2
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- added copper zone on F.Cu, net Net-(C6-Pad1)
Other:
- board size 56 x 61.5 mm -> 54.5 x 61.5 mm

Commit message: clean up pcb references and text
Parts:
- added G***: Panda, PandaLogos:Panda40x44mm, B.Cu at (76.5, 136.0)
Other:
- board text added: "IO"
- board text added: "Lightning"
- board text added: "NRF"
- board text added: "PGM"
- board text added: "PWR"
- board text added: "RESET"
- board text added: "RGB1"
- board text added: "RGB2"
- board text added: "RGB3"
- board text added: "RGB4"
- board text added: "S1"
- board text added: "S10"
- board text added: "S11"
- board text added: "S12"
- board text added: "S2"
- board text added: "S3"
- board text added: "S4"
- board text added: "S5"
- board text added: "S6"
- board text added: "S7"
- board text added: "S8"
- board text added: "S9"
- board text added: "Slave-V1"
- board text added: "Stock"

Commit message: updated pcb for prototype
Parts:
- added C10: 1µ, Capacitors_SMD:C_0603_HandSoldering, B.Cu at (97.8, 114.3)
- added C12: 1µ, Capacitors_SMD:C_0603_HandSoldering, B.Cu at (97.8, 116.8)
- added C13: 1µ, Capacitors_SMD:C_0603_HandSoldering, B.Cu at (97.8, 119.4)
- added C14: 1µ, Capacitors_SMD:C_0603_HandSoldering, B.Cu at (97.8, 131.8)
- added C15: 1µ, Capacitors_SMD:C_0603_HandSoldering, B.Cu at (97.8, 134.2)
- added C16: 1µ, Capacitors_SMD:C_0603_HandSoldering, B.Cu at (97.8, 136.8)
- added C17: 1µ, Capacitors_SMD:C_0603_HandSoldering, B.Cu at (97.8, 139.2)
- added C18: 1µ, Capacitors_SMD:C_0603_HandSoldering, B.Cu at (97.8, 151.8)
- added C19: 1µ, Capacitors_SMD:C_0603_HandSoldering, B.Cu at (97.8, 154.2)
- added C2: 1µ, Capacitors_SMD:C_0603_HandSoldering, B.Cu at (97.8, 111.8)
- added C20: 1µ, Capacitors_SMD:C_0603_HandSoldering, B.Cu at (97.8, 157.0)
- added C21: 1µ, Capacitors_SMD:C_0603_HandSoldering, B.Cu at (97.8, 159.5)
- added SW: SW_Push_SPDT, Pin_Headers:Pin_Header_Straight_1x03_Pitch2.54mm, F.Cu at (61.0, 108.0)
- J1: value Jack-DC -> 5V; footprint Connect:BARREL_JACK -> Pin_Headers:Pin_Header_Straight_1x02_Pitch2.54mm
- moved J1 8.51 mm to (56.0, 115.0), turned to 180 degrees
- moved C11 3.13 mm to (80.9, 113.1)
Connections:
- net Net-(C6-Pad1) renamed +5V
- D10 pad 2: +3V3 -> /Select array/Vdd
- D11 pad 2: +3V3 -> /Select array/Vdd
- D12 pad 2: +3V3 -> /Select array/Vdd
- D13 pad 2: +3V3 -> /Select array/Vdd
- D14 pad 2: +3V3 -> /Select array/Vdd
- D15 pad 2: +3V3 -> /Select array/Vdd
- D4 pad 2: +3V3 -> /Select array/Vdd
- D5 pad 2: +3V3 -> /Select array/Vdd
- D6 pad 2: +3V3 -> /Select array/Vdd
- D7 pad 2: +3V3 -> /Select array/Vdd
- D8 pad 2: +3V3 -> /Select array/Vdd
- D9 pad 2: +3V3 -> /Select array/Vdd
- Q1 pad 3: +3V3 -> /Select array/Vdd
- Q10 pad 3: +3V3 -> /Select array/Vdd
- Q11 pad 3: +3V3 -> /Select array/Vdd
- Q12 pad 3: +3V3 -> /Select array/Vdd
- Q2 pad 3: +3V3 -> /Select array/Vdd
- Q3 pad 3: +3V3 -> /Select array/Vdd
- Q4 pad 3: +3V3 -> /Select array/Vdd
- Q5 pad 3: +3V3 -> /Select array/Vdd
- Q6 pad 3: +3V3 -> /Select array/Vdd
- Q7 pad 3: +3V3 -> /Select array/Vdd
- Q8 pad 3: +3V3 -> /Select array/Vdd
- Q9 pad 3: +3V3 -> /Select array/Vdd
- R11 pad 1: +3V3 -> /Select array/Vdd
- R12 pad 1: +3V3 -> /Select array/Vdd
- R13 pad 1: +3V3 -> /Select array/Vdd
- R14 pad 1: +3V3 -> /Select array/Vdd
- R23 pad 1: +3V3 -> /Select array/Vdd
- R24 pad 1: +3V3 -> /Select array/Vdd
- R25 pad 1: +3V3 -> /Select array/Vdd
- R26 pad 1: +3V3 -> /Select array/Vdd
- R35 pad 1: +3V3 -> /Select array/Vdd
- R36 pad 1: +3V3 -> /Select array/Vdd
- R37 pad 1: +3V3 -> /Select array/Vdd
- R38 pad 1: +3V3 -> /Select array/Vdd
Routing:
- net +3V3: track 8.57 -> 13.8 mm, vias 2 -> 4
- net /Select array/S11: track 11.6 -> 14.4 mm
- net /Select array/S12: track 6.39 -> 9.24 mm
- net /Select array/S8: track 6.14 -> 8.99 mm
- net /Select array/S7: track 11.8 -> 14.6 mm
- net /Select array/S6: track 10.6 -> 13.4 mm
- net /Select array/S10: track 10.6 -> 13.4 mm
- net /Select array/S5: track 6.00 -> 8.80 mm
- net /Select array/S9: track 5.40 -> 8.20 mm
- net /Select array/S3: track 11.8 -> 14.5 mm
- net /Select array/S1: track 6.00 -> 8.77 mm
- net /Select array/S4: track 9.13 -> 11.9 mm
- net /Select array/S2: track 11.3 -> 14.0 mm
- net /NRF_CSN: track 18.1 -> 16.3 mm, vias 0 -> 1
- net /NRF_CE: track 15.4 -> 14.2 mm, vias 0 -> 1
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- added copper zone on F.Cu, net /Select array/Vdd
Other:
- board size 54.5 x 61.5 mm -> 51 x 61.5 mm
- board text added: "3.3V"
- board text added: "5V"
- board text added: "Gnd"
